File: 常用元器件库/reports/testboard/testboard.kicad_pcb (KiCad board)
At the start: 2 copper layers, 235 x 366.6 mm, 88 parts

Commit message: 直插化：6 条贴片件移到 _archive_smd_20261002；check_footprints 加禁止贴片规则并补自测
Co-Authored-By: Claude Opus 5.5 <noreply@anthropic.com>
Claude-Session: https://claude.ai/code/session_01FeFu9pjE12fFHg1a7J12km
Parts:
- removed Q-003: SOT-23, SOT-23
- removed REG-001: SOT-223-3_TabPin2, SOT-223-3_TabPin2
- removed REG-005: SOT-23-5, SOT-23-5
- removed USB-002: USB_C_Receptacle_ShouHan_TYPE-C-6P_PowerOnly, USB_C_Receptacle_ShouHan_TYPE-C-6P_PowerOnly
- removed USB-004: USB_C_Receptacle_HRO_TYPE-C-31-M-12, USB_C_Receptacle_HRO_TYPE-C-31-M-12
- moved XH-004 177.2 mm to (199.5, 333.6)
- moved XH-005 177.2 mm to (217.0, 333.6)
- moved XH-003 177.2 mm to (184.5, 333.6)
- moved CAP-004 175.2 mm to (195.1, 348.1)
- moved FUS-001 175.2 mm to (182.4, 348.2)
- moved LED-006 175.2 mm to (217.6, 347.9)
- moved Q-001 175.2 mm to (206.3, 348.4)
- moved CAP-001 61.6 mm to (98.9, 358.0)
- moved DIO-002 61.6 mm to (34.7, 358.1)
- moved DIO-004 61.6 mm to (51.8, 358.1)
- moved CAP-003 61.6 mm to (110.3, 358.0)
- moved DIO-001 61.6 mm to (121.5, 357.8)
- moved RES-001 61.6 mm to (68.6, 358.0)
- moved RES-002 61.6 mm to (82.4, 358.0)
- moved PH-006 52.5 mm to (110.3, 347.9)
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Other:
- board size 235 x 366.6 mm -> 235 x 365.7 mm
