File: 常用元器件库/reports/testboard/testboard.kicad_pcb (KiCad board)
At the start: 2 copper layers, 235 x 365.7 mm, 83 parts

Commit message: 第二批补完：Pico/Pico W/STC89C52RC/BlackPill/ESP32-CAM/LCD1602/I2C 转接板/LCD2004/TM1637/MAX7219/USB-TTL/ST-Link；离线模式；jlcparts 镜像导入工具
Co-Authored-By: Claude Opus 5.5 <noreply@anthropic.com>
Claude-Session: https://claude.ai/code/session_01FeFu9pjE12fFHg1a7J12km
Parts:
- added DSP-012: WC1602A, WC1602A, F.Cu at (155.6, 243.8)
- added DSP-013: PinHeader_1x04_P2.54mm_Vertical, PinHeader_1x04_P2.54mm_Vertical, F.Cu at (173.2, 362.5)
- added DSP-016: PinHeader_1x05_P2.54mm_Vertical, PinHeader_1x05_P2.54mm_Vertical, F.Cu at (202.8, 331.2)
- added MCU-012: RaspberryPi_Pico_Common_THT, RaspberryPi_Pico_Common_THT, F.Cu at (53.8, 183.8)
- added MCU-014: DIP-40_W15.24mm_Socket, DIP-40_W15.24mm_Socket, F.Cu at (134.9, 182.3)
- added MCU-015: Module_WeAct_BlackPill_STM32F411, Module_WeAct_BlackPill_STM32F411, F.Cu at (168.2, 313.3)
- added MCU-016: Module_ESP32-CAM_AiThinker, Module_ESP32-CAM_AiThinker, F.Cu at (33.4, 279.1)
- moved MCU-009 172.9 mm to (6.59, 245.2)
- moved DSP-003 137.2 mm to (80.6, 246.3)
- moved DSP-004 101.7 mm to (121.2, 246.3)
- moved DSP-006 64.7 mm to (11.6, 298.6)
- moved MCU-002 64.7 mm to (108.2, 314.3)
- moved DSP-001 64.7 mm to (47.8, 296.2)
- moved DSP-002 64.7 mm to (80.3, 296.2)
- moved SEG-003 49.6 mm to (158.0, 199.7)
- moved DSP-008 49.6 mm to (187.1, 185.4)
- moved SEG-001 47.7 mm to (210.9, 330.9)
- moved TERM-001 47.7 mm to (182.1, 366.4)
- moved TERM-002 47.7 mm to (197.2, 366.4)
- moved TERM-003 47.7 mm to (217.3, 366.4)
- moved BAT-002 47.1 mm to (43.6, 341.3)
- moved BZ-001 47.1 mm to (140.7, 367.0)
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Other:
- board size 235 x 365.7 mm -> 235 x 412.8 mm

Commit message: 第三批：69 条传感器/执行器/通信/电源模块（C 级为主，底板带脚名排针封装）；DS18B20、SRD 继电器取 GitHub 公开原版规格书
Co-Authored-By: Claude Opus 5.5 <noreply@anthropic.com>
Claude-Session: https://claude.ai/code/session_01FeFu9pjE12fFHg1a7J12km
Parts:
- added ACT-001: Module_Hdr_Relay_H_3P, Module_Hdr_Relay_H_3P, F.Cu at (60.9, 442.8)
- added ACT-002: Module_Hdr_Relay_L_3P, Module_Hdr_Relay_L_3P, F.Cu at (73.1, 442.8)
- added ACT-003: Relay_SPDT_SANYOU_SRD_Series_Form_C, Relay_SPDT_SANYOU_SRD_Series_Form_C, F.Cu at (162.2, 368.7)
- added ACT-004: Module_Hdr_SG90_3P, Module_Hdr_SG90_3P, F.Cu at (84.0, 442.8)
- added ACT-005: Module_Hdr_MG996R_3P, Module_Hdr_MG996R_3P, F.Cu at (95.8, 442.8)
- added ACT-006: Module_Hdr_ULN2003_6P, Module_Hdr_ULN2003_6P, F.Cu at (108.4, 364.4)
- added ACT-007: Module_Hdr_TB6612_8P, Module_Hdr_TB6612_8P, F.Cu at (111.3, 333.1)
- added ACT-008: Module_Hdr_L298N_7P, Module_Hdr_L298N_7P, F.Cu at (7.79, 364.4)
- added ACT-009: Module_Hdr_DRV8833_6P, Module_Hdr_DRV8833_6P, F.Cu at (120.7, 364.4)
- added ACT-010: Module_Hdr_DFPlayer_7P, Module_Hdr_DFPlayer_7P, F.Cu at (20.5, 364.4)
- added COM-001: Module_Hdr_HC-05_6P, Module_Hdr_HC-05_6P, F.Cu at (132.0, 364.4)
- added COM-002: Module_Hdr_HC-06_4P, Module_Hdr_HC-06_4P, F.Cu at (100.3, 409.0)
- added COM-003: Module_Hdr_ESP-01S_8P, Module_Hdr_ESP-01S_8P, F.Cu at (124.1, 333.1)
- added COM-004: PinSocket_2x04_P2.54mm_Vertical, PinSocket_2x04_P2.54mm_Vertical, F.Cu at (65.0, 424.3)
- added COM-005: Module_Hdr_MAX485_6P, Module_Hdr_MAX485_6P, F.Cu at (145.0, 364.4)
- added DSP-015: Module_Hdr_TM1637_4P, Module_Hdr_TM1637_4P, F.Cu at (115.3, 389.3)
- added SEN-001: Module_Hdr_DHT11_3P, Module_Hdr_DHT11_3P, F.Cu at (144.4, 426.2)
- added SEN-003: Module_Hdr_DHT22_4P, Module_Hdr_DHT22_4P, F.Cu at (126.7, 389.3)
- added SEN-004: Module_Hdr_AHT20_4P, Module_Hdr_AHT20_4P, F.Cu at (138.6, 389.3)
- added SEN-005: Module_Hdr_AHT20_BMP280_4P, Module_Hdr_AHT20_BMP280_4P, F.Cu at (153.1, 389.3)
- added SEN-006: Module_Hdr_SHT30_6P, Module_Hdr_SHT30_6P, F.Cu at (32.4, 364.4)
- added SEN-010: Module_Hdr_GY-906_4P, Module_Hdr_GY-906_4P, F.Cu at (166.3, 389.3)
- added SEN-011: Module_Hdr_MAX30102_7P, Module_Hdr_MAX30102_7P, F.Cu at (224.5, 333.1)
- added SEN-012: Module_Hdr_PulseSensor_3P, Module_Hdr_PulseSensor_3P, F.Cu at (159.1, 426.2)
- added SEN-013: Module_Hdr_AD8232_6P, Module_Hdr_AD8232_6P, F.Cu at (44.2, 364.4)
- added SEN-014: Module_Hdr_GY-521_8P, Module_Hdr_GY-521_8P, F.Cu at (75.2, 333.1)
- added SEN-015: Module_Hdr_GY-291_8P, Module_Hdr_GY-291_8P, F.Cu at (87.0, 333.1)
- added SEN-016: Module_Hdr_HC-SR501_3P, Module_Hdr_HC-SR501_3P, F.Cu at (172.7, 426.2)
- added SEN-017: Module_Hdr_AM312_3P, Module_Hdr_AM312_3P, F.Cu at (184.0, 426.2)
- added SEN-018: Module_Hdr_HC-SR04_4P, Module_Hdr_HC-SR04_4P, F.Cu at (178.5, 389.3)
- added SEN-019: Module_Hdr_HC-SR04P_4P, Module_Hdr_HC-SR04P_4P, F.Cu at (191.8, 389.3)
- added SEN-020: Module_Hdr_GY-530_6P, Module_Hdr_GY-530_6P, F.Cu at (57.8, 364.4)
- added SEN-021: Module_Hdr_RCWL-0516_5P, Module_Hdr_RCWL-0516_5P, F.Cu at (201.6, 364.4)
- added SEN-022: Module_Hdr_LD2410C_5P, Module_Hdr_LD2410C_5P, F.Cu at (213.9, 364.4)
- added SEN-025: Module_Hdr_GY-302_5P, Module_Hdr_GY-302_5P, F.Cu at (8.24, 389.3)
- added SEN-026: Module_Hdr_LDR_LM393_4P, Module_Hdr_LDR_LM393_4P, F.Cu at (205.6, 389.3)
- added SEN-027: Module_Hdr_Sound_4P, Module_Hdr_Sound_4P, F.Cu at (216.9, 389.3)
- added SEN-028: Module_Hdr_Flame_4P, Module_Hdr_Flame_4P, F.Cu at (7.79, 409.0)
- added SEN-029: Module_Hdr_Rain_4P, Module_Hdr_Rain_4P, F.Cu at (18.7, 409.0)
- added SEN-030: Module_Hdr_Soil_v1.2_3P, Module_Hdr_Soil_v1.2_3P, F.Cu at (197.2, 426.2)
- added SEN-031: Module_Hdr_WaterLevel_3P, Module_Hdr_WaterLevel_3P, F.Cu at (211.4, 426.2)
- added SEN-032: Module_Hdr_MQ-2_4P, Module_Hdr_MQ-2_4P, F.Cu at (29.6, 409.0)
- added SEN-033: Module_Hdr_MQ-135_4P, Module_Hdr_MQ-135_4P, F.Cu at (41.4, 409.0)
- added SEN-034: Module_Hdr_SW-420_3P, Module_Hdr_SW-420_3P, F.Cu at (223.7, 426.2)
- added SEN-035: Module_Hdr_TCRT5000_4P, Module_Hdr_TCRT5000_4P, F.Cu at (54.1, 409.0)
- added SEN-036: Module_Hdr_VS1838B_3P, Module_Hdr_VS1838B_3P, F.Cu at (8.70, 442.8)
- added SEN-037: Module_Hdr_KY-003_3P, Module_Hdr_KY-003_3P, F.Cu at (20.5, 442.8)
- added SEN-038: Module_Hdr_HX711_4P, Module_Hdr_HX711_4P, F.Cu at (65.4, 409.0)
- added SEN-039: Module_Hdr_ACS712_05B_3P, Module_Hdr_ACS712_05B_3P, F.Cu at (34.1, 442.8)
- added SEN-040: Module_Hdr_ACS712_20A_3P, Module_Hdr_ACS712_20A_3P, F.Cu at (48.2, 442.8)
- added SEN-041: Module_Hdr_INA219_4P, Module_Hdr_INA219_4P, F.Cu at (77.2, 409.0)
- added SEN-042: Module_Hdr_VSENSE25_2P, Module_Hdr_VSENSE25_2P, F.Cu at (209.6, 442.8)
- added SEN-043: Module_Hdr_ATGM336H_5P, Module_Hdr_ATGM336H_5P, F.Cu at (21.5, 389.3)
- added SEN-044: Module_Hdr_NEO-6M_4P, Module_Hdr_NEO-6M_4P, F.Cu at (89.0, 409.0)
- added SEN-045: Module_Hdr_RC522_8P, Module_Hdr_RC522_8P, F.Cu at (98.9, 333.1)
- added SEN-046: Module_Hdr_AS608_6P, Module_Hdr_AS608_6P, F.Cu at (70.3, 364.4)
- added SEN-047: Module_Hdr_DS3231_6P, Module_Hdr_DS3231_6P, F.Cu at (83.3, 364.4)
- added SEN-048: Module_Hdr_DS1302_5P, Module_Hdr_DS1302_5P, F.Cu at (33.3, 389.3)
- added SEN-049: Module_Hdr_MicroSD_6P, Module_Hdr_MicroSD_6P, F.Cu at (95.6, 364.4)
- DSP-013: value PinHeader_1x04_P2.54mm_Vertical -> Module_Hdr_PCF8574_LCD_I2C_4P; footprint PinHeader_1x04_P2.54mm_Vertical -> Module_Hdr_PCF8574_LCD_I2C_4P
- DSP-016: value PinHeader_1x05_P2.54mm_Vertical -> Module_Hdr_MAX7219_5P; footprint PinHeader_1x05_P2.54mm_Vertical -> Module_Hdr_MAX7219_5P
- moved SEG-001 143.9 mm to (78.4, 387.1)
- moved CAP-012 143.2 mm to (38.9, 457.1)
- moved SW-010 143.2 mm to (12.0, 457.6)
- moved XH-002 143.2 mm to (50.6, 456.6)
- moved XH-003 143.2 mm to (63.1, 456.6)
- moved XH-004 143.2 mm to (78.0, 456.6)
- moved XH-005 143.2 mm to (95.5, 456.6)
- moved SW-001 143.2 mm to (24.6, 455.2)
- moved PWR-001 136.9 mm to (67.9, 395.2)
- moved PWR-002 136.9 mm to (46.7, 387.1)
- moved DIO-002 132.9 mm to (152.3, 467.2)
- moved CAP-002 132.9 mm to (140.8, 467.5)
- moved DIO-004 132.9 mm to (169.3, 467.2)
- moved CAP-001 132.9 mm to (216.5, 467.1)
- moved DIO-005 132.9 mm to (124.0, 467.7)
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Other:
- board size 235 x 412.8 mm -> 235 x 483.3 mm
